File: kicad/AltairDrive.kicad_pcb (KiCad board)
At the start: 4 copper layers, 37 parts, among them J1 Conn_02x20_Odd_Even, J2 SERIAL, SW1 SW_Shutdown

Commit message: kicad files for front panel
Parts:
- removed SW1: SW_Shutdown, Connector_PinHeader_2.54mm:PinHeader_1x02_P2.54mm_Horizontal
- added J3: Conn_01x03_Pin, Connector:FanPinHeader_1x03_P2.54mm_Vertical, B.Cu at (77.6, 63.1)
- added J4: I2C, Connector:FanPinHeader_1x04_P2.54mm_Vertical, B.Cu at (212.1, 79.5)
- added SW2: SW_PWR, MrEppot:E-Switch, F.Cu at (73.3, 87.4)
- added SW3: SW_RBT, MrEppot:E-Switch, F.Cu at (88.3, 87.3)
- J1: moved to B.Cu
- J2: footprint Connector_PinHeader_2.54mm:PinHeader_2x05_P2.54mm_Horizontal -> Connector:FanPinHeader_1x03_P2.54mm_Vertical; moved to B.Cu
- moved J2 308.3 mm to (195.7, 63.1), turned to 180 degrees
- moved D13 301.3 mm to (222.7, 88.6)
- moved D14 301.3 mm to (237.7, 88.6)
- moved R13 301.2 mm to (222.7, 67.7)
- moved D10 300.7 mm to (222.7, 128.6)
- moved D11 300.7 mm to (237.7, 128.6)
- moved D12 300.7 mm to (252.7, 128.6)
- moved R10 300.7 mm to (222.7, 106.4)
- moved R11 300.7 mm to (237.7, 106.4)
- moved R12 300.7 mm to (252.7, 106.4)
- moved D15 300.3 mm to (252.7, 88.6)
- moved R14 300.2 mm to (237.7, 67.4)
- moved R15 300.2 mm to (252.7, 67.4)
- moved D7 295.7 mm to (167.7, 128.6)
- moved D8 295.7 mm to (182.7, 128.6)
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Connections:
- J1 pad 12: unconnected-(J1-Pin_12-Pad12) -> Net-(J1-Pin_12)
- J1 pad 19: unconnected-(J1-Pin_19-Pad19) -> Net-(J1-Pin_19)
- J1 pad 21: unconnected-(J1-Pin_21-Pad21) -> Net-(J1-Pin_21)
- J1 pad 23: unconnected-(J1-Pin_23-Pad23) -> Net-(J1-Pin_23)
- J1 pad 32: unconnected-(J1-Pin_32-Pad32) -> Net-(J1-Pin_32)
- J1 pad 39: Net-(J1-Pin_39) -> unconnected-(J1-Pin_39-Pad39)
- J1 pad 4: Net-(J1-Pin_4) -> unconnected-(J1-Pin_4-Pad4)
- J1 pad 5: unconnected-(J1-Pin_5-Pad5) -> Net-(J1-Pin_5)
- J1 pad 7: Net-(J1-Pin_7) -> unconnected-(J1-Pin_7-Pad7)
- J2 pad 1: unconnected-(J2-Pin_1-Pad1) -> Net-(D1-K)
- J2 pad 2: unconnected-(J2-Pin_2-Pad2) -> Net-(J1-Pin_8)
- J2 pad 3: unconnected-(J2-Pin_3-Pad3) -> Net-(J1-Pin_10)
- R1 pad 1: Net-(J1-Pin_11) -> Net-(J1-Pin_12)
- R10 pad 1: Net-(J1-Pin_35) -> Net-(J1-Pin_31)
- R11 pad 1: Net-(J1-Pin_37) -> Net-(J1-Pin_29)
- R12 pad 1: Net-(J1-Pin_39) -> Net-(J1-Pin_23)
- R13 pad 1: Net-(J1-Pin_36) -> Net-(J1-Pin_21)
- R14 pad 1: Net-(J1-Pin_38) -> Net-(J1-Pin_19)
- R15 pad 1: Net-(J1-Pin_40) -> Net-(J1-Pin_15)
- R16 pad 1: Net-(J1-Pin_2) -> Net-(J1-Pin_22)
- R17 pad 1: Net-(J1-Pin_7) -> Net-(J1-Pin_40)
- R2 pad 1: Net-(J1-Pin_13) -> Net-(J1-Pin_16)
- R3 pad 1: Net-(J1-Pin_15) -> Net-(J1-Pin_18)
- R4 pad 1: Net-(J1-Pin_16) -> Net-(J1-Pin_32)
- R5 pad 1: Net-(J1-Pin_18) -> Net-(J1-Pin_36)
- R6 pad 1: Net-(J1-Pin_22) -> Net-(J1-Pin_38)
- R7 pad 1: Net-(J1-Pin_29) -> Net-(J1-Pin_37)
- R8 pad 1: Net-(J1-Pin_31) -> Net-(J1-Pin_35)
Routing:
- net Net-(D1-K): track 0.00 -> 576.2 mm
- net Net-(J1-Pin_13): track 0.00 -> 159.5 mm
- net Net-(J1-Pin_11): track 0.00 -> 156.5 mm
- net Net-(J1-Pin_12): track 0.00 -> 144.1 mm
- net Net-(J1-Pin_16): track 0.00 -> 122.2 mm
- net Net-(J1-Pin_15): track 0.00 -> 120.6 mm
- net Net-(J1-Pin_22): track 0.00 -> 119.7 mm
- net Net-(J1-Pin_19): track 0.00 -> 111.0 mm
- net Net-(J1-Pin_18): track 0.00 -> 108.4 mm
- net Net-(J1-Pin_23): track 0.00 -> 104.4 mm
- net Net-(J1-Pin_29): track 0.00 -> 97.7 mm
- net Net-(J1-Pin_21): track 0.00 -> 94.8 mm
- net Net-(J1-Pin_31): track 0.00 -> 85.9 mm
- net Net-(J1-Pin_33): track 0.00 -> 64.8 mm
- net Net-(J1-Pin_32): track 0.00 -> 63.3 mm
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Other:
- board outline added: 207 x 76 mm
- copper layers 4 -> 2
- board text added: "DP-A REV-1 2025 MR EPPOT"
- board text added: "I2C"
- board text added: "PWR"
- board text added: "SERIAL"
- board text removed: "ALTAIR DISK SERVER (C)2025 MREPPOT"
